Commit message: Updated URDF Limits to +- 180

File: canadarm2_description/urdf/CanadaArm2-DAE-ROS2.urdf (robot description, URDF)
Before this commit: robot CanadaArm2, 8 links, 7 joints
Joints:
- joint joint_1: limit lower=0.0 upper=6.283185 effort=100 velocity=100 -> lower=-3.141593 upper=3.141593 effort=100 velocity=100
- joint joint_2: limit lower=0.0 upper=6.283185 effort=100 velocity=100 -> lower=-3.141593 upper=3.141593 effort=100 velocity=100
- joint joint_3: limit lower=0.0 upper=6.283185 effort=100 velocity=100 -> lower=-3.141593 upper=3.141593 effort=100 velocity=100
- joint joint_4: limit lower=0.0 upper=6.283185 effort=100 velocity=100 -> lower=-3.141593 upper=3.141593 effort=100 velocity=100
- joint joint_5: limit lower=0.0 upper=6.283185 effort=100 velocity=100 -> lower=-3.141593 upper=3.141593 effort=100 velocity=100
- joint joint_6: limit lower=0.0 upper=6.283185 effort=100 velocity=100 -> lower=-3.141593 upper=3.141593 effort=100 velocity=100
- joint joint_7: limit lower=0.0 upper=6.283185 effort=100 velocity=100 -> lower=-3.141593 upper=3.141593 effort=100 velocity=100

File: canadarm2_description/urdf/CanadaArm2-DAE.urdf (robot description, URDF)
Before this commit: robot CanadaArm2, 8 links, 7 joints
Joints:
- joint joint_1: limit lower=0.0 upper=6.283185 effort=100 velocity=100 -> lower=-3.141593 upper=3.141593 effort=100 velocity=100
- joint joint_2: limit lower=0.0 upper=6.283185 effort=100 velocity=100 -> lower=-3.141593 upper=3.141593 effort=100 velocity=100
- joint joint_3: limit lower=0.0 upper=6.283185 effort=100 velocity=100 -> lower=-3.141593 upper=3.141593 effort=100 velocity=100
- joint joint_4: limit lower=0.0 upper=6.283185 effort=100 velocity=100 -> lower=-3.141593 upper=3.141593 effort=100 velocity=100
- joint joint_5: limit lower=0.0 upper=6.283185 effort=100 velocity=100 -> lower=-3.141593 upper=3.141593 effort=100 velocity=100
- joint joint_6: limit lower=0.0 upper=6.283185 effort=100 velocity=100 -> lower=-3.141593 upper=3.141593 effort=100 velocity=100
- joint joint_7: limit lower=0.0 upper=6.283185 effort=100 velocity=100 -> lower=-3.141593 upper=3.141593 effort=100 velocity=100

File: canadarm2_description/urdf/CanadaArm2-OBJ-ROS2.urdf (robot description, URDF)
Before this commit: robot CanadaArm2, 8 links, 7 joints
Joints:
- joint joint_1: limit lower=0.0 upper=6.283185 effort=100 velocity=100 -> lower=-3.141593 upper=3.141593 effort=100 velocity=100
- joint joint_2: limit lower=0.0 upper=6.283185 effort=100 velocity=100 -> lower=-3.141593 upper=3.141593 effort=100 velocity=100
- joint joint_3: limit lower=0.0 upper=6.283185 effort=100 velocity=100 -> lower=-3.141593 upper=3.141593 effort=100 velocity=100
- joint joint_4: limit lower=0.0 upper=6.283185 effort=100 velocity=100 -> lower=-3.141593 upper=3.141593 effort=100 velocity=100
- joint joint_5: limit lower=0.0 upper=6.283185 effort=100 velocity=100 -> lower=-3.141593 upper=3.141593 effort=100 velocity=100
- joint joint_6: limit lower=0.0 upper=6.283185 effort=100 velocity=100 -> lower=-3.141593 upper=3.141593 effort=100 velocity=100
- joint joint_7: limit lower=0.0 upper=6.283185 effort=100 velocity=100 -> lower=-3.141593 upper=3.141593 effort=100 velocity=100

File: canadarm2_description/urdf/CanadaArm2-OBJ.urdf (robot description, URDF)
Before this commit: robot CanadaArm2, 8 links, 7 joints
Joints:
- joint joint_1: limit lower=0.0 upper=6.283185 effort=100 velocity=100 -> lower=-3.141593 upper=3.141593 effort=100 velocity=100
- joint joint_2: limit lower=0.0 upper=6.283185 effort=100 velocity=100 -> lower=-3.141593 upper=3.141593 effort=100 velocity=100
- joint joint_3: limit lower=0.0 upper=6.283185 effort=100 velocity=100 -> lower=-3.141593 upper=3.141593 effort=100 velocity=100
- joint joint_4: limit lower=0.0 upper=6.283185 effort=100 velocity=100 -> lower=-3.141593 upper=3.141593 effort=100 velocity=100
- joint joint_5: limit lower=0.0 upper=6.283185 effort=100 velocity=100 -> lower=-3.141593 upper=3.141593 effort=100 velocity=100
- joint joint_6: limit lower=0.0 upper=6.283185 effort=100 velocity=100 -> lower=-3.141593 upper=3.141593 effort=100 velocity=100
- joint joint_7: limit lower=0.0 upper=6.283185 effort=100 velocity=100 -> lower=-3.141593 upper=3.141593 effort=100 velocity=100

File: canadarm2_description/urdf/CanadaArm2-PLY-ROS2.urdf (robot description, URDF)
Before this commit: robot CanadaArm2, 8 links, 7 joints
Joints:
- joint joint_1: limit lower=0.0 upper=6.283185 effort=100 velocity=100 -> lower=-3.141593 upper=3.141593 effort=100 velocity=100
- joint joint_2: limit lower=0.0 upper=6.283185 effort=100 velocity=100 -> lower=-3.141593 upper=3.141593 effort=100 velocity=100
- joint joint_3: limit lower=0.0 upper=6.283185 effort=100 velocity=100 -> lower=-3.141593 upper=3.141593 effort=100 velocity=100
- joint joint_4: limit lower=0.0 upper=6.283185 effort=100 velocity=100 -> lower=-3.141593 upper=3.141593 effort=100 velocity=100
- joint joint_5: limit lower=0.0 upper=6.283185 effort=100 velocity=100 -> lower=-3.141593 upper=3.141593 effort=100 velocity=100
- joint joint_6: limit lower=0.0 upper=6.283185 effort=100 velocity=100 -> lower=-3.141593 upper=3.141593 effort=100 velocity=100
- joint joint_7: limit lower=0.0 upper=6.283185 effort=100 velocity=100 -> lower=-3.141593 upper=3.141593 effort=100 velocity=100

File: canadarm2_description/urdf/CanadaArm2-PLY.urdf (robot description, URDF)
Before this commit: robot CanadaArm2, 8 links, 7 joints
Joints:
- joint joint_1: limit lower=0.0 upper=6.283185 effort=100 velocity=100 -> lower=-3.141593 upper=3.141593 effort=100 velocity=100
- joint joint_2: limit lower=0.0 upper=6.283185 effort=100 velocity=100 -> lower=-3.141593 upper=3.141593 effort=100 velocity=100
- joint joint_3: limit lower=0.0 upper=6.283185 effort=100 velocity=100 -> lower=-3.141593 upper=3.141593 effort=100 velocity=100
- joint joint_4: limit lower=0.0 upper=6.283185 effort=100 velocity=100 -> lower=-3.141593 upper=3.141593 effort=100 velocity=100
- joint joint_5: limit lower=0.0 upper=6.283185 effort=100 velocity=100 -> lower=-3.141593 upper=3.141593 effort=100 velocity=100
- joint joint_6: limit lower=0.0 upper=6.283185 effort=100 velocity=100 -> lower=-3.141593 upper=3.141593 effort=100 velocity=100
- joint joint_7: limit lower=0.0 upper=6.283185 effort=100 velocity=100 -> lower=-3.141593 upper=3.141593 effort=100 velocity=100

File: canadarm2_description/urdf/CanadaArm2-ROS2.urdf (robot description, URDF)
Before this commit: robot CanadaArm2, 8 links, 7 joints
Joints:
- joint joint_1: limit lower=0.0 upper=6.283185 effort=100 velocity=100 -> lower=-3.141593 upper=3.141593 effort=100 velocity=100
- joint joint_2: limit lower=0.0 upper=6.283185 effort=100 velocity=100 -> lower=-3.141593 upper=3.141593 effort=100 velocity=100
- joint joint_3: limit lower=0.0 upper=6.283185 effort=100 velocity=100 -> lower=-3.141593 upper=3.141593 effort=100 velocity=100
- joint joint_4: limit lower=0.0 upper=6.283185 effort=100 velocity=100 -> lower=-3.141593 upper=3.141593 effort=100 velocity=100
- joint joint_5: limit lower=0.0 upper=6.283185 effort=100 velocity=100 -> lower=-3.141593 upper=3.141593 effort=100 velocity=100
- joint joint_6: limit lower=0.0 upper=6.283185 effort=100 velocity=100 -> lower=-3.141593 upper=3.141593 effort=100 velocity=100
- joint joint_7: limit lower=0.0 upper=6.283185 effort=100 velocity=100 -> lower=-3.141593 upper=3.141593 effort=100 velocity=100

File: canadarm2_description/urdf/CanadaArm2.urdf (robot description, URDF)
Before this commit: robot CanadaArm2, 8 links, 7 joints
Joints:
- joint joint_1: limit lower=0.0 upper=6.283185 effort=100 velocity=100 -> lower=-3.141593 upper=3.141593 effort=100 velocity=100
- joint joint_2: limit lower=0.0 upper=6.283185 effort=100 velocity=100 -> lower=-3.141593 upper=3.141593 effort=100 velocity=100
- joint joint_3: limit lower=0.0 upper=6.283185 effort=100 velocity=100 -> lower=-3.141593 upper=3.141593 effort=100 velocity=100
- joint joint_4: limit lower=0.0 upper=6.283185 effort=100 velocity=100 -> lower=-3.141593 upper=3.141593 effort=100 velocity=100
- joint joint_5: limit lower=0.0 upper=6.283185 effort=100 velocity=100 -> lower=-3.141593 upper=3.141593 effort=100 velocity=100
- joint joint_6: limit lower=0.0 upper=6.283185 effort=100 velocity=100 -> lower=-3.141593 upper=3.141593 effort=100 velocity=100
- joint joint_7: limit lower=0.0 upper=6.283185 effort=100 velocity=100 -> lower=-3.141593 upper=3.141593 effort=100 velocity=100
